File: hardware/v0.2/robot_board.brd (EAGLE design)
At the start: 95.2 x 76.1 mm, 161 parts, among them J1 POWER_JACKPTH, Q1 DMP2035U, Q2 DMP2035U, Q3 DMP2035U-7, Q4 DMP2035U-7, U1 FT232RL-BASICSSOP, U10 DRV8839, U12 LM393, U16 LM393, U17 ATMEGA325PA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

Commit message: fix servo code
Parts:
- R36: value 600K 1% -> 604K 1%
- R39, R43, R63, R65: value 1K -> 1K 1%
- R44: value 100K -> 100K 1%
- R45, R46: value 10K 1% -> 100K 1%
- R53: value 1.5K -> 1.5K 1%
Changed lines of the file:
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@@
 <element name="U16" library="SparkFun-AnalogIC" package="SO08" value="LM393" x="81.6356" y="17.7546" rot="R270"/>
 <element name="R35" library="resistor" package="R1206" value="120K 1%" x="82.2706" y="22.0726"/>
-<element name="R36" library="resistor" package="R1206" value="600K 1%" x="82.2452" y="24.638" rot="R180"/>
+<element name="R36" library="resistor" package="R1206" value="604K 1%" x="82.2452" y="24.638" rot="R180"/>
 <element name="JP8" library="SparkFun-Connectors" package="2X3" value="" x="64.77" y="63.5"/>
-<element name="R39" library="resistor" package="R1206" value="1K" x="69.6214" y="58.8264" rot="R90"/>
+<element name="R39" library="resistor" package="R1206" value="1K 1%" x="69.6214" y="58.8264" rot="R90"/>
 <element name="R41" library="resistor" package="R1206" value="330" x="3.81" y="66.1924" rot="R180"/>
 <element name="D25" library="SparkFun-LED" package="LED-1206" value="POWER" x="2.5146" y="61.722" rot="R90">
@@
 <attribute name="NAME" x="95.123" y="15.2908" size="0.508" layer="25" font="vector" rot="R270"/>
 </element>
-<element name="R43" library="resistor" package="R1206" value="1K" x="87.4014" y="10.6934" smashed="yes" rot="R270">
+<element name="R43" library="resistor" package="R1206" value="1K 1%" x="87.4014" y="10.6934" smashed="yes" rot="R270">
 <attribute name="NAME" x="84.9884" y="13.8684" size="1.27" layer="25" rot="R270"/>
 <attribute name="VALUE" x="84.9884" y="12.0904" size="1.27" layer="27" rot="R270"/>
 </element>
-<element name="R44" library="resistor" package="R1206" value="100K" x="88.4936" y="18.796" rot="R270"/>
+<element name="R44" library="resistor" package="R1206" value="100K 1%" x="88.4936" y="18.796" rot="R270"/>
 <element name="U$19" library="r_cubed" package="2POS_TERMINAL" value="2POS_TERMINAL" x="32.3596" y="70.6882" rot="R180"/>
 <element name="U$20" library="r_cubed" package="2POS_TERMINAL" value="2POS_TERMINAL" x="22.352" y="70.6882" rot="R180"/>
-<element name="R45" library="resistor" package="R1206" value="10K 1%" x="52.832" y="26.8986"/>
-<element name="R46" library="resistor" package="R1206" value="10K 1%" x="53.3654" y="22.1996" rot="R90"/>
+<element name="R45" library="resistor" package="R1206" value="100K 1%" x="52.832" y="26.8986"/>
+<element name="R46" library="resistor" package="R1206" value="100K 1%" x="53.3654" y="22.1996" rot="R90"/>
 <element name="U1" library="SparkFun-DigitalIC" package="SSOP28DB" value="FT232RL-BASICSSOP" x="49.784" y="6.35" rot="R270"/>
 <element name="R47" library="resistor" package="R1206" value="300" x="9.398" y="63.246" smashed="yes" rot="R90">
@@
 <element name="R52" library="resistor" package="R1206" value="330" x="9.144" y="4.572" rot="R90"/>
 <element name="U8" library="jseng" package="SOT23-M5" value="MIC2009A" x="65.659" y="42.4434" smashed="yes" rot="R90"/>
-<element name="R53" library="resistor" package="R1206" value="1.5K" x="66.04" y="47.1678" smashed="yes" rot="R180">
+<element name="R53" library="resistor" package="R1206" value="1.5K 1%" x="66.04" y="47.1678" smashed="yes" rot="R180">
 <attribute name="NAME" x="66.675" y="49.5808" size="1.27" layer="25" rot="R180"/>
 <attribute name="VALUE" x="67.437" y="49.5808" size="1.27" layer="27" rot="R180"/>
@@
 <element name="C8" library="resistor" package="C1206" value=".1uF" x="49.53" y="40.386" rot="R270"/>
 <element name="C9" library="resistor" package="C1206" value="1uF" x="63.8556" y="55.3212" rot="R90"/>
-<element name="R63" library="resistor" package="R1206" value="1K" x="53.2892" y="14.6304" rot="R90"/>
+<element name="R63" library="resistor" package="R1206" value="1K 1%" x="53.2892" y="14.6304" rot="R90"/>
 <element name="U$2" library="r_cubed" package="POT" value="POT" x="36.0172" y="2.7686"/>
 <element name="D34" library="SparkFun-LED" package="LED-1206" value="RX" x="42.4434" y="3.7846" rot="R270">
 <attribute name="PROD_ID" value="DIO-09910" x="42.4434" y="3.7846" size="1.016" layer="27" font="vector" rot="R270" display="off"/>
 </element>
-<element name="R65" library="resistor" package="R1206" value="1K" x="68.7578" y="43.307" rot="R270"/>
+<element name="R65" library="resistor" package="R1206" value="1K 1%" x="68.7578" y="43.307" rot="R270"/>
 <element name="D24" library="diode" package="SOT23" value="BAT54C" x="73.8124" y="30.4546"/>
 <element name="R28" library="resistor" package="R1206" value="1M" x="59.309" y="37.6682" rot="R270"/>
